File: hardware/unit-board/can_main_interface.kicad_sch (KiCad schematic)
At the start: 8 parts, among them J4 SM03B-GHS-TB, J5 SM03B-GHS-TB, SW2 JS102011SAQN, U5 TCAN1051VDRQ1

Commit message: fix(hardware): resolve unit board ERC violations
Parts:
- removed J5: SM03B-GHS-TB, Connector_JST:JST_GH_SM03B-GHS-TB_1x03-1MP_P1.25mm_Horizontal, symbol Connector_Generic:Conn_01x03
- added J3: SM03B-GHS-TB, Connector_JST:JST_GH_SM03B-GHS-TB_1x03-1MP_P1.25mm_Horizontal, symbol Connector_Generic:Conn_01x03
- renumbered C17 to C1, C18 to C2, D2 to D1, J4 to J2, R5 to R1, SW2 to SW1, U5 to U3
Connections:
- net GND: now also J3.3 (Pin_3)
- net C620_CAN_H renamed COMM_A
- net COMM_A: now also J3.1 (Pin_1)
- net C620_CAN_L renamed COMM_B
- net COMM_B: now also J3.2 (Pin_2)
