File: hardware/unit-board/power_3v3.kicad_sch (KiCad schematic)
At the start: 8 parts, among them J1 SM02B-GHS-TB, U1 LM66100DCKR, U2 TLV1117LV33DCYR

Commit message: fix(hardware): resolve unit board ERC violations
Connections:
- net GND: now also J1.2 (Pin_2); no longer J1.1 (Pin_1)
- net PWR_5V: now reaches C201.1, C202.1, U1.3 (~{CE}), U1.6 (VOUT), U2.3 (VI)
- net PWR_5V_IN: now reaches C101.1, U1.1 (VIN)
- net PWR_5V_IN: now also J1.1 (Pin_1); no longer J1.2 (Pin_2)
- net +3.3V renamed 3.3V
- no-connect marks 0 -> 1
Changed lines of the file:
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@@
 	(generator_version "10.0")
 	(paper "A4")
+	(symbol
+		(lib_id "power:PWR_FLAG")
+		(at 58.42 85.09 0)
+		(unit 1)
+		(body_style 1)
+		(exclude_from_sim no)
+		(in_bom yes)
+		(on_board yes)
+		(in_pos_files yes)
+		(dnp no)
+		(property "Reference" "#FLG01" (at 58.42 87.63 0) (hide yes) (effects (font (size 1.27 1.27))))
+		(property "Value" "PWR_FLAG" (at 58.42 88.9 0) (effects (font (size 1.27 1.27))))
+		(property "Footprint" "" (at 58.42 85.09 0) (hide yes) (effects (font (size 1.27 1.27))))
+		(property "Datasheet" "" (at 58.42 85.09 0) (hide yes) (effects (font (size 1.27 1.27))))
+		(property "Description" "Special symbol for telling ERC where power comes from" (at 58.42 85.09 0) (hide yes) (effects (font (size 1.27 1.27))))
+		(pin "1")
+		(instances (project "unit-board" (path "/902d1696-b686-472b-a104-e0c03f0522c9/a7bf357a-460b-4605-a722-18c5392efee3" (reference "#FLG01") (unit 1))))
+	)
+	(symbol
+		(lib_id "power:PWR_FLAG")
+		(at 46.99 93.98 0)
+		(unit 1)
+		(body_style 1)
+		(exclude_from_sim no)
+		(in_bom yes)
+		(on_board yes)
+		(in_pos_files yes)
+		(dnp no)
+		(property "Reference" "#FLG02" (at 46.99 96.52 0) (hide yes) (effects (font (size 1.27 1.27))))
+		(property "Value" "PWR_FLAG" (at 46.99 97.79 0) (effects (font (size 1.27 1.27))))
+		(property "Footprint" "" (at 46.99 93.98 0) (hide yes) (effects (font (size 1.27 1.27))))
+		(property "Datasheet" "" (at 46.99 93.98 0) (hide yes) (effects (font (size 1.27 1.27))))
+		(property "Description" "Special symbol for telling ERC where power comes from" (at 46.99 93.98 0) (hide yes) (effects (font (size 1.27 1.27))))
+		(pin "1")
+		(instances (project "unit-board" (path "/902d1696-b686-472b-a104-e0c03f0522c9/a7bf357a-460b-4605-a722-18c5392efee3" (reference "#FLG02") (unit 1))))
+	)
+	(no_connect
+		(at 109.22 87.63)
+	)
 	(junction
 		(at 121.92 85.09)
@@
 	(wire
 		(pts
-			(xy 194.31 85.09) (xy 199.39 85.09)
+			(xy 194.31 85.09) (xy 201.93 85.09)
 		)
 		(stroke
@@
 	(wire
 		(pts
+			(xy 114.3 77.47) (xy 116.84 77.47)
+		)
+		(stroke
+			(width 0)
+			(type default)
+		)
+	)
+	(wire
+		(pts
 			(xy 134.62 88.9) (xy 134.62 85.09)
 		)
@@
 	(wire
 		(pts
-			(xy 46.99 85.09) (xy 58.42 85.09)
+			(xy 46.99 87.63) (xy 58.42 87.63)
+		)
+		(stroke
+			(width 0)
+			(type default)
+		)
+	)
+	(wire
+		(pts
+			(xy 58.42 87.63) (xy 58.42 85.09)
 		)
 		(stroke
@@
 	(wire
 		(pts
-			(xy 46.99 87.63) (xy 46.99 93.98)
+			(xy 46.99 85.09) (xy 44.45 85.09)
+		)
+		(stroke
+			(width 0)
+			(type default)
+		)
+	)
+	(wire
+		(pts
+			(xy 44.45 85.09) (xy 44.45 93.98)
+		)
+		(stroke
+			(width 0)
+			(type default)
+		)
+	)
+	(wire
+		(pts
+			(xy 44.45 93.98) (xy 46.99 93.98)
 		)
 		(stroke
@@
 	(wire
 		(pts
+			(xy 114.3 85.09) (xy 114.3 77.47)
+		)
+		(stroke
+			(width 0)
+			(type default)
+		)
+	)
+	(wire
+		(pts
 			(xy 134.62 85.09) (xy 147.32 85.09)
 		)
@@
 			(width 0)
 			(type default)
+		)
+	)
+	(label "PWR_5V_IN"
+		(at 58.42 85.09 0)
+		(effects
+			(font
+				(size 1.27 1.27)
+			)
+			(justify left bottom)
+		)
+	)
+	(hierarchical_label "PWR_5V"
+		(shape output)
+		(at 116.84 77.47 0)
+		(effects
+			(font
+				(size 1.27 1.27)
+			)
+			(justify left)
+		)
+	)
+	(hierarchical_label "3.3V"
+		(shape output)
+		(at 201.93 85.09 0)
+		(effects
+			(font
+				(size 1.27 1.27)
+			)
+			(justify left)
 		)
 	)
@@
 					(unit 1)
 				)
-			)
-		)
-	)
-	(symbol
-		(lib_id "power:+3.3V")
-		(at 199.39 85.09 270)
-		(unit 1)
-		(body_style 1)
-		(exclude_from_sim no)
-		(in_bom yes)
-		(on_board yes)
-		(in_pos_files yes)
-		(dnp no)
-		(fields_autoplaced yes)
-		(property "Reference" "#PWR09"
-			(at 195.58 85.09 0)
-			(hide yes)
-			(show_name no)
-			(do_not_autoplace no)
-			(effects
-				(font
-					(size 1.27 1.27)
-				)
-			)
-		)
-		(property "Value" "+3.3V"
-			(at 203.2 85.0899 90)
-			(show_name no)
-			(do_not_autoplace no)
-			(effects
-				(font
-					(size 1.27 1.27)
-				)
-				(justify left)
-			)
-		)
-		(property "Footprint" ""
-			(at 199.39 85.09 0)
-			(hide yes)
-			(show_name no)
-			(do_not_autoplace no)
-			(effects
-				(font
-					(size 1.27 1.27)
-				)
-			)
-		)
-		(property "Datasheet" ""
-			(at 199.39 85.09 0)
-			(hide yes)
-			(show_name no)
-			(do_not_autoplace no)
-			(effects
-				(font
-					(size 1.27 1.27)
-				)
-			)
-		)
-		(property "Description" "Power symbol creates a global label with name \"+3.3V\""
-			(at 199.39 85.09 0)
-			(hide yes)
-			(show_name no)
-			(do_not_autoplace no)
-			(effects
-				(font
-					(size 1.27 1.27)
-				)
-			)
-		)
-		(pin "1"
-		)
-		(instances
-			(project "unit-board"
-				(path "/902d1696-b686-472b-a104-e0c03f0522c9/a7bf357a-460b-4605-a722-18c5392efee3"
-					(reference "#PWR09")
-					(unit 1)
-				)
