File: hardware/unit-board/unit-board.kicad_pcb (KiCad board)
At the start: 4 copper layers, 45 x 45 mm, 64 parts, among them J1 SM02B-GHS-TB, J2 SM03B-GHS-TB, J3 SM03B-GHS-TB, J4 SM03B-GHS-TB, J5 SM03B-GHS-TB, J6 SM06B-GHS-TB, J7 BM06B-GHS-TBT, SW1 JS102011SAQN, SW3 A6S-3104-H, U1 LM66100DCKR, U2 TLV1117LV33DCYR, U3 TCAN1051VDRQ1, U4 STM32G474RET6, U5 TCAN1051VDRQ1, Y1 ECS-80-8-33Q-JES-TR

Commit message: chore: update CAD and finalize unit board layout
Parts:
- removed ? (x2): , 
- removed the REF** at (97.0, 58.0)
- removed the REF** at (58.0, 58.0)
- added REF**: MountingHole_2.7mm_M2.5, MountingHole:MountingHole_2.7mm_M2.5, F.Cu at (97.0, 58.0)
- added REF**: MountingHole_2.7mm_M2.5, MountingHole:MountingHole_2.7mm_M2.5, F.Cu at (97.0, 97.0)
- added REF**: MountingHole_2.7mm_M2.5, MountingHole:MountingHole_2.7mm_M2.5, F.Cu at (58.0, 97.0)
- added REF**: MountingHole_2.7mm_M2.5, MountingHole:MountingHole_2.7mm_M2.5, F.Cu at (58.0, 58.0)
- moved J4 38.6 mm to (96.8, 65.1), turned to 90 degrees
- moved J5 38.5 mm to (58.4, 65.1), turned to -90 degrees
- moved R1 22.2 mm to (90.8, 86.9), turned to 180 degrees
- moved D6 20.7 mm to (72.9, 93.2), turned to 0 degrees
- moved SW1 20.0 mm to (87.4, 93.5)
- moved R19 19.2 mm to (72.8, 91.8), turned to 0 degrees
- moved C6 18.5 mm to (70.7, 85.2), turned to 0 degrees
- moved D8 18.1 mm to (67.4, 62.1)
- moved R20 15.3 mm to (68.9, 62.1)
- moved C1 15.2 mm to (72.0, 88.2), turned to 90 degrees
- moved D9 15.1 mm to (61.7, 85.8), turned to 90 degrees
- moved D10 13.3 mm to (63.7, 85.8), turned to 90 degrees
- moved C204 13.2 mm to (80.1, 82.7), turned to 180 degrees
- moved C203 13.1 mm to (80.1, 80.9), turned to 180 degrees
- moved R21 12.9 mm to (61.7, 82.8), turned to -90 degrees
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Routing:
- net /CAN Interface/3.3V: track 0.00 -> 218.0 mm, vias 0 -> 9
- net GND: track 0.00 -> 83.3 mm, vias 0 -> 54
- net /CAN Interface/PWR_5V: track 0.97 -> 83.0 mm, vias 0 -> 4
- net /CAN Interface/COMM_A: track 15.9 -> 60.5 mm, vias 0 -> 2
- net /G474 Minimum/UNIT_ID2: track 0.00 -> 38.8 mm, vias 0 -> 2
- net /CAN Interface1/CAN_RX: track 0.00 -> 37.1 mm, vias 0 -> 2
- net /CAN Interface1/C620_CAN_H: track 11.5 -> 47.9 mm, vias 0 -> 2
- net /G474 Minimum/UNIT_ID1: track 0.00 -> 35.0 mm, vias 0 -> 2
- net /CAN Interface1/CAN_TX: track 0.00 -> 32.7 mm, vias 0 -> 2
- net /CAN Interface/COMM_B: track 14.8 -> 47.1 mm, vias 0 -> 2
- net /G474 Minimum/UNIT_ID0: track 0.00 -> 30.9 mm, vias 0 -> 2
- net /CAN Interface1/C620_CAN_L: track 12.3 -> 42.3 mm, vias 0 -> 2
- net /G474 Minimum/ADC_5V_MON: track 0.12 -> 27.7 mm, vias 0 -> 2
- net /G474 Minimum/NRST: track 0.00 -> 26.0 mm, vias 0 -> 2
- net /G474 Minimum/AMT22_CS_N: track 0.00 -> 18.9 mm, vias 0 -> 2
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- added copper zone on In1.Cu, net GND
