File: hardware/unit-board/unit-board.kicad_pcb (KiCad board)
At the start: 4 copper layers, 45 x 45 mm, 64 parts, among them J1 SM02B-GHS-TB, J2 SM03B-GHS-TB, J3 SM03B-GHS-TB, J4 SM03B-GHS-TB, J5 SM03B-GHS-TB, J6 SM06B-GHS-TB, J7 BM06B-GHS-TBT, SW1 JS102011SAQN, SW3 A6S-3104-H, U1 LM66100DCKR, U2 TLV1117LV33DCYR, U3 TCAN1051VDRQ1, U4 STM32G474RET6, U5 TCAN1051VDRQ1, Y1 ECS-80-8-33Q-JES-TR

Commit message: Resolve odometry board ERC and finalize unit board CAD outputs
- AMT102 encoder input buffers: consolidate the per-channel 74LVC2G17
  from 2 parts (one gate each, power unit unplaced) into 1 part using
  all 3 units (gate A + gate B + power), wired to GND/PWR_3.3V. Fixes
  the remaining 18 ERC violations; odometry board schematic is now
  0 errors / 0 warnings across all sheets.
- Add odometry board schematic reference doc, block-diagram figures,
  and schematic+BOM HTML/PDF exports.
- Add DifferentialSwerve logo library (footprint + symbol) referenced
  by the schematics.
- Finalize unit board layout/CAD and commit fabrication outputs
  (Gerbers, drill report, JLCPCB BOM, STEP model).
- Ignore tmp/ (scratch working directory; can contain automation
  browser profiles with login data and must never be committed).

Co-Authored-By: Claude Sonnet 5 <noreply@anthropic.com>
Parts:
- added G***: LOGO, DifferentialSwerve:DifferentialSwerve_Logo, F.Cu at (66.0, 64.0)
- added QR*****: QR_GitHub_Repository, QR_GitHub_Repository, F.Cu at (64.6, 84.0)
Other:
- board text added: "1"
- board text added: "120Ω"
- board text added: "2"
- board text added: "4"
- board text added: "5V_IN"
- board text added: "CAN1"
- board text added: "CAN2"
- board text added: "COM"
- board text added: "DIFFERENTIAL SWERVE UNIT CONTROLLER STM32G474 • DUAL CAN • C620 x2 • AMT22 5V INPUT • 3.3V LOGIC CENTRAL CAN / MOTOR CAN UNIT ID: 1 / 2 / 4 REV.A"
- board text added: "ERR"
- board text added: "H"
- board text added: "ID"
- board text added: "ON"
- board text added: "PWR"
- board text added: "RUN"
- board text added: "△"
