File: hardware/unit-board/unit-board.kicad_pcb (KiCad board)
At the start: 4 copper layers, 45 x 45 mm, 66 parts, among them J1 SM02B-GHS-TB, J2 SM03B-GHS-TB, J3 SM03B-GHS-TB, J4 SM03B-GHS-TB, J5 SM03B-GHS-TB, J6 SM06B-GHS-TB, J7 BM06B-GHS-TBT, SW1 JS102011SAQN, SW3 A6S-3104-H, U1 LM66100DCKR, U2 TLV1117LV33DCYR, U3 TCAN1051VDRQ1, U4 STM32G474RET6, U5 TCAN1051VDRQ1, Y1 ECS-80-8-33Q-JES-TR

Commit message: Update project design and manufacturing artifacts
Parts:
- D7: value BAT54SLT1G -> BAT54S-HF
- R13: value RC0603FR-0733KL 33k -> RC0603FR-0722KL 22k
- R14: value RC0603FR-0722KL 22k -> RC0603FR-0710KL 10k
- SW3: value A6S-3104-H -> DS04-254-1-03BK-SMT
- U2: value TLV1117LV33DCYR -> TLV76133DCYR
- Y1: value ECS-80-8-33Q-JES-TR -> FC3BAEBDI8.0-T1
Changed lines of the file:
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@@
 			)
 		)
-		(property "Value" "RC0603FR-0722KL 22k"
+		(property "Value" "RC0603FR-0710KL 10k"
 			(at 0 1.43 90)
 			(layer "F.Fab")
@@
 			)
 		)
-		(property "Value" "TLV1117LV33DCYR"
+		(property "Value" "TLV76133DCYR"
 			(at 0 4.500001 0)
 			(layer "F.Fab")
@@
 			)
 		)
-		(property "Value" "RC0603FR-0733KL 33k"
+		(property "Value" "RC0603FR-0722KL 22k"
 			(at 0 1.43 90)
 			(layer "F.Fab")
@@
 			)
 		)
-		(property "Value" "ECS-80-8-33Q-JES-TR"
+		(property "Value" "FC3BAEBDI8.0-T1"
 			(at 0 2.450001 0)
 			(layer "F.Fab")
@@
 			)
 		)
-		(property "Value" "A6S-3104-H"
+		(property "Value" "DS04-254-1-03BK-SMT"
 			(at 0 5.34 90)
 			(layer "F.Fab")
@@
 			)
 		)
-		(property "Value" "BAT54SLT1G"
+		(property "Value" "BAT54S-HF"
 			(at 0 2.4 0)
 			(layer "F.Fab")
