File: hardware/odometry-board/Oddom board/Oddom board.kicad_sch (KiCad schematic)
At the start: 37 parts, among them J1 SM02B-GHS-TB, J7 Conn_01x08, J8 BM06B-GHS-TBT, SW3 A6S-3104-H, U1 LM66100DCKR, U1 STM32F405RGTx, U2 TLV1117LV33DCYR, Y1 ECS-80-8-33Q-JES-TR

Commit message: WIP: place odometry board footprints
Parts:
- renumbered U1 to U5
Connections:
- net PWR_5V: now also C2.1, C3.1, U2.3 (VI), U5.6 (VOUT)

Commit message: WIP: route odometry board RevA
Parts:
- added C27: 2.2 µF, Capacitor_SMD:C_0805_2012Metric, symbol Device:C
- added C28: 100nF, Capacitor_SMD:C_0603_1608Metric, symbol Device:C
Connections:
- net GND: now also C27.2, C28.1
- net PWR_3.3V: now also C27.1, C28.2
Other:
- moved on the sheet: J7
