File: hardware/odometry-board/Oddom board/Oddom board.kicad_pcb (KiCad board)
At the start: 2 copper layers, 65 x 27.5 mm, 69 parts, among them J1 SM02B-GHS-TB, J2 SM03B-GHS-TB, J4 Conn_01x04, J5 Conn_01x04, J6 Conn_01x04, J7 Conn_01x08, J8 BM06B-GHS-TBT, SW1 JS102011SAQN, SW3 A6S-3104-H, U1 STM32F405RGTx, U2 TLV1117LV33DCYR, U3 74LVC2G17, U4 TCAN1051VDRQ1, U5 LM66100DCKR, U7 74LVC2G17, U9 74LVC2G17, Y1 ECS-80-8-33Q-JES-TR

Commit message: WIP: route odometry board RevA
Parts:
- moved C14 10.7 mm to (99.7, 95.5), turned to 0 degrees
- moved C11 8.97 mm to (96.7, 98.8), turned to -90 degrees
- moved C24 6.86 mm to (78.0, 98.4), turned to 90 degrees
- moved D3 5.43 mm to (71.6, 95.0)
- moved R7 4.97 mm to (75.7, 93.9), turned to 0 degrees
- moved C7 4.59 mm to (101.8, 102.6), turned to 0 degrees
- moved C23 4.58 mm to (76.3, 98.5), turned to 90 degrees
- moved R6 3.89 mm to (75.7, 95.6), turned to 0 degrees
- moved R3 3.62 mm to (101.8, 97.6), turned to 180 degrees
- moved C25 3.02 mm to (106.9, 96.7)
- moved R8 3.02 mm to (106.9, 98.2)
- moved C26 2.97 mm to (106.9, 95.2)
- moved R9 2.97 mm to (106.9, 93.8)
- moved C22 1.57 mm to (96.7, 95.5)
- moved REF** 1.00 mm to (128.5, 100.0)
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Routing:
- net PWR_3.3V: track 0.00 -> 183.9 mm, vias 0 -> 10
- net PWR_5V: track 0.00 -> 104.3 mm, vias 0 -> 2
- net GND: track 0.00 -> 76.3 mm, vias 0 -> 46
- net SWDIO: track 0.00 -> 49.9 mm, vias 0 -> 2
- net SWCLK: track 0.00 -> 49.7 mm, vias 0 -> 2
- net IMU_INT1: track 0.00 -> 46.7 mm, vias 0 -> 1
- net Net-(J7-Pin_3): track 0.00 -> 44.9 mm, vias 0 -> 1
- net IMU_INT2: track 0.00 -> 42.3 mm, vias 0 -> 1
- net Net-(J7-Pin_4): track 0.00 -> 39.2 mm, vias 0 -> 1
- net Net-(U1-PC6): track 0.00 -> 36.5 mm, vias 0 -> 2
- net Net-(U1-PC8): track 0.00 -> 35.6 mm, vias 0 -> 2
- net Net-(U1-PC7): track 0.00 -> 35.6 mm, vias 0 -> 2
- net Net-(J7-Pin_5): track 0.00 -> 34.6 mm, vias 0 -> 1
- net USART2_RX: track 0.00 -> 34.2 mm, vias 0 -> 2
- net IMU_CS_N: track 0.00 -> 32.9 mm, vias 0 -> 1
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- added copper zone on In1.Cu, net GND
Other:
- copper layers 2 -> 4

Commit message: Finalize odometry board silkscreen and fabrication outputs
Parts:
- added G***: LOGO, DifferentialSwerve:DifferentialSwerve_Logo, F.Cu at (119.9, 107.8)
- added QR*****: git@github.com:Posaka-Y/Differential-Swerve-Drive.git, git@github.com:Posaka-Y/Differential-Swerve-Drive.git, F.Cu at (83.3, 99.8)
Routing:
- net GND: vias 46 -> 45
Other:
- board text added: "CAN"
- board text added: "COM"
- board text added: "DIFFERENTIAL SWERVE ODOMETRY F405 REV.A UNIT ID:4 CAN 1Mbps"
- board text added: "ERR"
- board text added: "H"
- board text added: "ID0 ID1 ID2"
- board text added: "IMU"
- board text added: "OFF ON"
- board text added: "PWR"
- board text added: "RUN"
- board text added: "△"

Commit message: Update project design and manufacturing artifacts
Parts:
- SW3: value A6S-3104-H -> DS04-254-1-03BK-SMT
- U2: value TLV1117LV33DCYR -> TLV76133DCYR
- Y1: value ECS-80-8-33Q-JES-TR -> FC3BAEBDI8.0-T1
Changed lines of the file:
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@@
 			)
 		)
-		(property "Value" "TLV1117LV33DCYR"
+		(property "Value" "TLV76133DCYR"
 			(at 0 4.500001 0)
 			(layer "F.Fab")
@@
 			)
 		)
-		(property "Value" "ECS-80-8-33Q-JES-TR"
+		(property "Value" "FC3BAEBDI8.0-T1"
 			(at 0.3 3.4 0)
 			(layer "F.Fab")
@@
 			)
 		)
-		(property "Value" "A6S-3104-H"
+		(property "Value" "DS04-254-1-03BK-SMT"
 			(at 0 5.34 0)
 			(layer "F.Fab")
