File: hardware/odometry-board/5V monitoring.kicad_sch (KiCad schematic)
At the start: 4 parts

Commit message: Update project design and manufacturing artifacts
Parts:
- D7: value BAT54S -> BAT54S-HF
Changed lines of the file:
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@@
 			)
 		)
-		(property "Value" "BAT54S"
+		(property "Value" "BAT54S-HF"
 			(at 136.144 50.8 90)
 			(show_name no)
