File: hardware/central-board-placement/S02B_star_teensy-1.kicad_sch (KiCad schematic)
At the start: 41 parts, among them J201 SM02B-GHS-TB, J202 SM02B-GHS-TB, J203 SM02B-GHS-TB, J204 SM02B-GHS-TB, J210 Teensy 4.1 socket, SW211 REARM switch TBD

Commit message: Save all current circuit, firmware, CAD and manufacturing work
Parts:
- removed C212: 100nF, Capacitor_SMD:C_0603_1608Metric, symbol Device:C
- removed D201, D202, D203, D204, D205, D206: LTST-C190KGKT, LED_SMD:LED_0603_1608Metric, symbol Device:LED
- removed F201, F202, F203, F204, F206: 1206L050/15YR, Fuse:Fuse_1206_3216Metric, symbol Device:Polyfuse
- removed F205: 1206L075/16YR, Fuse:Fuse_1206_3216Metric, symbol Device:Polyfuse
- removed J201, J202, J203, J204: SM02B-GHS-TB, Connector_JST:JST_GH_SM02B-GHS-TB_1x02-1MP_P1.25mm_Horizontal, symbol Connector_Generic:Conn_01x02
- removed R201, R202, R203, R204, R205, R206: 1.5k, Resistor_SMD:R_0603_1608Metric, symbol Device:R
- removed TP211: +5V_UNIT1, DifferentialSwerve:Harwin_S1751-46R, symbol Connector:TestPoint
- removed TP212: +5V_UNIT2, DifferentialSwerve:Harwin_S1751-46R, symbol Connector:TestPoint
- removed TP213: +5V_UNIT3, DifferentialSwerve:Harwin_S1751-46R, symbol Connector:TestPoint
- added C211: 100nF, Capacitor_SMD:C_0603_1608Metric, symbol Device:C
- J210: Placement note 単一48pinは旧J210/J211の代替。列中心間15.24mm、pad順は転記資料3.2。socket実物/ドリル照合は未完了; socket contacts are passive; firmware signal directions are separate design data -> 単一48pinは旧J210/J211の代替。列中心間15.24mm、pad順は転記資料3.2。socket実物/ドリル照合は未完了; socket contacts are passive; firmware signal directions are separate design data; pad11/pin9=PWR_USB_FAULT_N (2026-09-26 proposal), pad36/pin14 remains NC
- R214: Placement note (none) -> Local tactile ARM request; shared Teensy gate with GUI ARM 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
- SW211: Placement note 型番/基板またはパネル配置未確定 -> Local tactile ARM request; shared Teensy gate with GUI ARM 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
- renumbered C211 to C212
Connections:
- net REARM_SW_N: now reaches R214.1
- net REARM_SW_N: now also J210.8 (6), SW211.1, C211.1
- net +3V3_TEENSY: now reaches R214.2
- net +3V3_TEENSY: now also C212.1, J210.15 (3.3V), J210.46 (3.3V), TP217.1
- net GND_CTRL: now reaches D212.1 (K)
- net GND_CTRL: now also C212.2, D211.1 (K), D213.1 (K), J210.1 (GND), J210.34 (GND), J210.47 (GND), SW211.2, TP218.1, C211.2
- net at D212.2 (A): now also R212.1
- net +5V_ODOM: now reaches TP214.1
- net +5V_EXP: now reaches TP216.1
- net +5V_TEENSY_F: now reaches TP215.1
- net +5V_SYS: now reaches R213.1
- net at R213.2: now also D213.2 (A)
- net STATUS_G_LED: now reaches R211.1
- net STATUS_G_LED: now also J210.9 (7)
- net at R211.2: now also D211.2 (A)
- net STATUS_R_LED: now reaches R212.2
- net STATUS_R_LED: now also J210.10 (8)
- net PWR_USB_FAULT_N: now reaches J210.11 (9)
- net SPI_CS0_N: now reaches J210.12 (10)
- net SPI_MOSI: now reaches J210.13 (11)
- net SPI_MISO: now reaches J210.14 (12)
- net IO24_A10: now reaches J210.16 (24/A10)
- net IO25_A11: now reaches J210.17 (25/A11)
- net IO26_A12: now reaches J210.18 (26/A12)
- net IO27_A13: now reaches J210.19 (27/A13)
- net CAN2_RX: now reaches J210.2 (0)
- net UART7_RX: now reaches J210.20 (28)
- net UART7_TX: now reaches J210.21 (29)
- net CAN3_RX: now reaches J210.22 (30)
- net CAN3_TX: now reaches J210.23 (31)
- net PWR_5V_FAULT_N: now reaches J210.24 (32)
- net UART8_RX: now reaches J210.26 (34)
- net UART8_TX: now reaches J210.27 (35)
- net SPI_CS1_N: now reaches J210.28 (36)
- net CAN2_TX: now reaches J210.3 (1)
- net IO40_A16: now reaches J210.32 (40/A16)
- net IO41_A17: now reaches J210.33 (41/A17)
- net SPI_SCK: now reaches J210.35 (13)
- net I2C1_SCL: now reaches J210.38 (16/A2)
- net I2C1_SDA: now reaches J210.39 (17/A3)
- net MOTOR_PWR_EN: now reaches J210.4 (2)
- net I2C0_SDA: now reaches J210.40 (18/A4)
- net I2C0_SCL: now reaches J210.41 (19/A5)
- net IO20_A6: now reaches J210.42 (20/A6)
- net IO21_A7: now reaches J210.43 (21/A7)
- net CAN1_TX: now reaches J210.44 (22/A8)
- net CAN1_RX: now reaches J210.45 (23/A9)
- net VIN_TEENSY: now reaches J210.48 (VIN)
- net ESTOP_LOOP_OK_N: now reaches J210.5 (3)
- no-connect marks 0 -> 8
Other:
- note added: "ARM REQUESTS (2026-09-26) GUI on robot display -> mini PC USB-CDC -> Teensy shared ARM decision. SW211 tactile -> REARM_SW_N (pad8 / GPIO6) -> SAME decision; local maintenance. R214 10k pull-up to +3V3_TEENSY; C211 100nF to GND; SW211 to GND. E-stop release alone / held button / old GUI request never re-arms. ARM: MOTOR_PWR_EN ON, motion ZERO. Separate NEW RUN required. Teensy USB/GPIO adapter an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"
- note added: "GPIO PURPOSE LABELS | socket pad numbers differ from GPIO numbers GPIO4/5: reserved (individual E-stop monitor removed) GPIO9 / pad11: USB fault allocation PROPOSED Other RESERVED / NC pins are intentionally unconnected"
- note added: "GPIO14/A0 RESERVED / NC"
- note added: "GPIO15/A1 RESERVED / NC"
- note added: "GPIO33 RESERVED / NC"
- note added: "GPIO37 RESERVED / NC"
- note added: "GPIO38 RESERVED / NC"
- note added: "GPIO39 RESERVED / NC"
- note added: "GPIO4 RESERVED / NC"
- note added: "GPIO5 RESERVED / NC"
- note removed: "Footprint TBD"
- note removed: "PLACEMENT ONLY - all pins intentionally unwired; see notes in symbol properties."
- note removed: "REVIEW"
- note removed: "Star power / Teensy / indicators (1)"
- note removed: "UNRESOLVED: COMM LED - GPIO / implementation / reference pending."
- title: Star power / Teensy / indicators (1) -> Teensy 4.1 / REARM / RUN ERR PWR indicators
- moved on the sheet: C212, D211, D212, D213, R211, R212, R213, R214, SW211
