File: hardware/central-board-placement/S04_safety-1.kicad_sch (KiCad schematic)
At the start: 33 parts, among them J401 43650-0600, J402 TBD 2pin, J403 TBD 2pin, Q401 IRLML0100TRPBF, U401 LTV-847S, U402 SN74AHCT1G125DBVR

Commit message: Save all current circuit, firmware, CAD and manufacturing work
Parts:
- removed D402, D403, D404: 1N4148W, Diode_SMD:D_SOD-123, symbol Diode:1N4148W
- removed J401: 43650-0600, Connector_Molex:Molex_Micro-Fit_3.0_43650-0600_1x06_P3.00mm_Horizontal, symbol Connector_Generic:Conn_01x06
- removed R403, R404, R405, R406, R407, R408: 2.2k, Resistor_SMD:R_0603_1608Metric, symbol Device:R
- removed R410, R411, R412: 10k, Resistor_SMD:R_0603_1608Metric, symbol Device:R
- removed TP402: ESTOP1_AUX_OK_N, TestPoint:TestPoint_Pad_D1.5mm, symbol Connector:TestPoint
- removed TP403: ESTOP2_AUX_OK_N, TestPoint:TestPoint_Pad_D1.5mm, symbol Connector:TestPoint
- removed TP404: SPARE_24V_IN, TestPoint:TestPoint_Pad_D1.5mm, symbol Connector:TestPoint
- removed TP405: SPARE_OK_N, TestPoint:TestPoint_Pad_D1.5mm, symbol Connector:TestPoint
- removed unit 4 of U401
- removed unit 3 of U401
- removed unit 2 of U401
- added D405: SMBJ33CA, Diode_SMD:D_SMB, symbol Device:D_TVS
- added F402: TBD LED branch fuse, symbol Device:Fuse
- added J401: TBD E-stop 4pin, symbol Connector_Generic:Conn_01x04
- added X402: RETURN JOIN TBD, symbol CentralPlacement:ReturnJoin_TBD
- C401: Placement note U402 bypass, PDF candidate -> Connected schematic; see nonpower wiring review 2026-09-29
- D401, R401, R402, R409: Placement note (none) -> Connected schematic; see nonpower wiring review 2026-09-29
- F401: Placement note 定格/型番/配置未確定 -> Connected schematic; see nonpower wiring review 2026-09-29
- J402: Placement note 暫定1=COIL_POS / 2=COIL_NEG; 正式MPN/pin順/key未確定 -> Connected schematic; see nonpower wiring review 2026-09-29
- J403: footprint (none) -> Connector_JST:JST_XH_S2B-XH-A_1x02_P2.50mm_Horizontal; Placement note 暫定1=24V_CTRL_IN / 2=GND_24V_RETURN; 正式MPN/pin順/key未確定 -> Connected schematic; see nonpower wiring review 2026-09-29
- Q401: Placement note 2026-09-23 PDF基本案:1=G 2=S 3=D -> Connected schematic; see nonpower wiring review 2026-09-29
- R413: Placement note Input pulldown, PDF candidate -> Connected schematic; see nonpower wiring review 2026-09-29
- R414: Placement note Gate resistor, PDF candidate -> Connected schematic; see nonpower wiring review 2026-09-29
- R415: Placement note Gate pulldown, PDF candidate -> Connected schematic; see nonpower wiring review 2026-09-29
- TP401, TP406: Placement note Signal pad -> Connected schematic; see nonpower wiring review 2026-09-29
- U401: value LTV-847S -> LTV-817S; footprint (none) -> Package_DIP:SMDIP-4_W9.53mm; symbol Isolator:LTV-847S -> Isolator:LTV-817S; Placement note 4 units all required. footprint未確定; SMDIP-16_W9.53mm候補を実物照合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 -> Connected schematic; see nonpower wiring review 2026-09-29
- U402: Placement note 2026-09-23 PDF候補、DBV:1=OE_N 2=A 3=GND 4=Y 5=VCC。symbol pin要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 -> Connected schematic; see nonpower wiring review 2026-09-29
Connections:
- net COIL_BUFFER_OUT: now reaches R414.1
- net COIL_BUFFER_OUT: now also U402.4
- net COIL_GATE: now reaches R414.2
- net COIL_GATE: now also Q401.1 (G), R415.1
- net ESTOP_LOOP_RETURN: now reaches J402.1 (Pin_1)
- net ESTOP_LOOP_RETURN: now also R401.1, D405.1 (A1), J401.2 (Pin_2)
- net COIL_NEG: now reaches J402.2 (Pin_2)
- net COIL_NEG: now also Q401.3 (D), D405.2 (A2)
- net +3V3_TEENSY: now reaches R409.1
- net ESTOP_LOOP_OK_N: now reaches R409.2
- net ESTOP_LOOP_OK_N: now also TP401.1, U401.4
- net +5V_SYS: now reaches C401.1
- net +5V_SYS: now also U402.5 (VCC)
- net GND_CTRL: now reaches C401.2
- net GND_CTRL: now also R413.2, U401.3, U402.1, U402.3 (GND), X402.1 (LOGIC)
- net GND_24V_RETURN: now reaches Q401.2 (S)
- net GND_24V_RETURN: now also J403.2 (Pin_2), R415.2, X402.3 (COIL)
- net MONITOR_LED_A: now reaches D401.1 (K)
- net MONITOR_LED_A: now also R402.2, U401.1
- net GND_CTRL_LED: now reaches D401.2 (A)
- net GND_CTRL_LED: now also TP406.1, U401.2, J401.4 (Pin_4), X402.2 (LED)
- net MON_R: now reaches R402.1
- net MON_R: now also R401.2
- net MOTOR_PWR_EN: now reaches U402.2
- net MOTOR_PWR_EN: now also R413.1
- net +24V_CTRL_IN: now reaches F401.1
- net +24V_CTRL_IN: now also J403.1 (Pin_1), F402.1
- net ESTOP_LOOP_OUT: now reaches F401.2
- net ESTOP_LOOP_OUT: now also J401.1 (Pin_1)
- new net ESTOP_LED_24V: F402.2, J401.3 (Pin_3)
Other:
- note added: "24 V LOOP & EXTERNAL CONNECTORS"
- note added: "5 V BUFFER -> 100 V MOSFET / DEFAULT OFF"
- note added: "D405: SMBJ33CA / BIDIRECTIONAL / 33 V Release time and surge energy: bench verification pending"
- note added: "E-STOP LOOP / COIL DRIVER"
- note added: "F401 / F402: current rating, breaking capacity and footprints TBD LED measurement: 24 V / ~0.3 W (~12.5 mA); quantity not confirmed"
- note added: "J401: 1 OUT -> NC1 11-12 -> NC2 11-12 -> 2 RETURN 3 LED supply -> X1/X2 (polarity verify); 4 LED return Buttons / contactor are external to this board."
- note added: "NC LOOP MONITOR (LOW = LOOP ENERGIZED)"
- note added: "R401 + R402 = 4.4k total. D401 is reverse-parallel with optocoupler LED. Loop indication does not verify main contact opening / welding."
- note added: "Unresolved: J401/J402/J403 selection; F401/F402; X402 return connection. D405 selected; release time / transient validation pending. Not for fabrication."
- note added: "X402 is an unresolved return-connection interface, NOT a conductive net tie. Join location / routing must be resolved before hardware use. Driver requires a defined logic-to-coil return reference."
- note removed: "E-stop monitoring / central coil driver (1)"
- note removed: "Footprint TBD"
- note removed: "PLACEMENT ONLY - all pins intentionally unwired; see notes in symbol properties."
- note removed: "REVIEW"
- note removed: "UNRESOLVED: D4xx coil clamp - topology / polarity / rating / part pending."
- note removed: "UNRESOLVED: LED branch protection - F402 / rating / part pending."
- title: E-stop monitoring / central coil driver (1) -> E-stop NC loop monitor / coil driver / explicit TBD interfaces
- moved on the sheet: C401, D401, F401, J402, J403, Q401, R401, R402, R409, R413, R414, R415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
