File: hardware/central-board-placement/S05_io-1.kicad_sch (KiCad schematic)
At the start: 43 parts, among them J501 SM04B-GHS-TB, J502 SM04B-GHS-TB, J503 SM04B-GHS-TB, J504 SM03B-GHS-TB, J505 SM03B-GHS-TB, J506 SM07B-GHS-TB, J507 SM10B-GHS-TB, U501 SRV05-4, U502 SRV05-4, U503 SRV05-4, U504 SRV05-4, U505 SRV05-4, U506 SRV05-4

Commit message: Save all current circuit, firmware, CAD and manufacturing work
Parts:
- added J508, J509, J510: SM04B-GHS-TB, Connector_JST:JST_GH_SM04B-GHS-TB_1x04-1MP_P1.25mm_Horizontal, symbol Connector_Generic:Conn_01x04
- added JP505: GPIO VCC 3V3/5V select, Connector_PinHeader_2.54mm:PinHeader_1x03_P2.54mm_Vertical, symbol Connector_Generic:Conn_01x03
- J501, J502, J503, J504, J505, J506, JP501, JP502, JP503, JP504, R511, R512, R513, R514, R521, R522, R523, R524, R531, R532, R533, R534, R535, R541, R542, R543, R544, R545, R546, R547, R548, R551, R552, R553, R554: Placement note (none) -> Connected schematic; see nonpower wiring review 2026-09-29
- J507: value SM10B-GHS-TB -> SM04B-GHS-TB; footprint Connector_JST:JST_GH_SM10B-GHS-TB_1x10-1MP_P1.25mm_Horizontal -> Connector_JST:JST_GH_SM04B-GHS-TB_1x04-1MP_P1.25mm_Horizontal; symbol Connector_Generic:Conn_01x10 -> Connector_Generic:Conn_01x04; Placement note J507 GH10 format/pin order proposal -> Connected schematic; see nonpower wiring review 2026-09-29
- TP501: Placement note S1751-46R -> Connected schematic; see nonpower wiring review 2026-09-29
- U501, U502, U503, U504, U505, U506: Placement note Manufacturer not fixed; pin1/3/4/6=IO,2=GND,5=3V3; verify l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 -> Connected schematic; see nonpower wiring review 2026-09-29
Connections:
- net I2C0_SDA: now reaches R511.1
- net I2C0_SDA: now also R551.2
- net I2C0_SDA_EXT: now reaches R511.2
- net I2C0_SDA_EXT: now also J501.2 (Pin_2), J502.3 (Pin_3), U501.1 (IO1)
- net +3V3_TEENSY: now reaches JP502.1 (A)
- net +3V3_TEENSY: now also J502.1 (Pin_1), J503.1 (Pin_1), J506.1 (Pin_1), JP501.1 (A), JP503.1 (A), JP504.1 (A), U501.5 (VP), U502.5 (VP), U503.5 (VP), U504.5 (VP), U505.5 (VP), U506.5 (VP), JP505.1 (Pin_1)
- net PU_I2C0_SCL: now reaches JP502.2 (B)
- net PU_I2C0_SCL: now also R552.1
- net SPI_CS1_N_EXT: now reaches U504.1 (IO1)
- net SPI_CS1_N_EXT: now also J506.7 (Pin_7), R535.2
- net GND_CTRL: now reaches U504.2 (VN)
- net GND_CTRL: now also J501.1 (Pin_1), J502.2 (Pin_2), J503.2 (Pin_2), J504.1 (Pin_1), J505.1 (Pin_1), J506.2 (Pin_2), J507.2 (Pin_2), TP501.1, U501.2 (VN), U502.2 (VN), U503.2 (VN), U505.2 (VN), U506.2 (VN), J508.2 (Pin_2), J509.2 (Pin_2), J510.2 (Pin_2)
- net PU_I2C0_SDA: now reaches JP501.2 (B)
- net PU_I2C0_SDA: now also R551.1
- net I2C0_SCL_EXT: now reaches U501.3 (IO2)
- net I2C0_SCL_EXT: now also J501.3 (Pin_3), J502.4 (Pin_4), R512.2
- net I2C1_SDA_EXT: now reaches U501.4 (IO3)
- net I2C1_SDA_EXT: now also J503.3 (Pin_3), R513.2
- net I2C1_SCL_EXT: now reaches U501.6 (IO4)
- net I2C1_SCL_EXT: now also J503.4 (Pin_4), R514.2
- net SPI_SCK: now reaches R531.1
- net SPI_SCK_EXT: now reaches R531.2
- net SPI_SCK_EXT: now also J506.3 (Pin_3), U503.1 (IO1)
- net I2C1_SDA: now reaches R513.1
- net I2C1_SDA: now also R553.2
- net UART7_TX_EXT: now reaches U502.1 (IO1)
- net UART7_TX_EXT: now also J504.2 (Pin_2), R521.2
- net UART7_RX_EXT: now reaches U502.3 (IO2)
- net UART7_RX_EXT: now also J504.3 (Pin_3), R522.2
- net UART8_TX_EXT: now reaches U502.4 (IO3)
- net UART8_TX_EXT: now also J505.2 (Pin_2), R523.2
- net UART8_RX_EXT: now reaches U502.6 (IO4)
- net UART8_RX_EXT: now also J505.3 (Pin_3), R524.2
- net IO26_A12_EXT: now reaches U506.1 (IO1)
- net IO26_A12_EXT: now also R545.2, J509.3 (Pin_3)
- net IO27_A13_EXT: now reaches U506.3 (IO2)
- net IO27_A13_EXT: now also R546.2, J509.4 (Pin_4)
- net IO40_A16_EXT: now reaches U506.4 (IO3)
- net IO40_A16_EXT: now also R547.2, J510.3 (Pin_3)
- net IO41_A17_EXT: now reaches U506.6 (IO4)
- net IO41_A17_EXT: now also R548.2, J510.4 (Pin_4)
- net SPI_CS1_N: now reaches R535.1
- net I2C1_SCL: now reaches R514.1
- net I2C1_SCL: now also R554.2
- net I2C0_SCL: now reaches R512.1
- net I2C0_SCL: now also R552.2
- net IO41_A17: now reaches R548.1
- net PU_I2C1_SDA: now reaches JP503.2 (B)
- net PU_I2C1_SDA: now also R553.1
- net PU_I2C1_SCL: now reaches JP504.2 (B)
- net PU_I2C1_SCL: now also R554.1
- net UART8_TX: now reaches R523.1
- net SPI_CS0_N: now reaches R534.1
- net SPI_CS0_N_EXT: now reaches R534.2
- net SPI_CS0_N_EXT: now also J506.6 (Pin_6), U503.6 (IO4)
- net IO20_A6: now reaches R541.1
- net IO20_A6_EXT: now reaches R541.2
- net IO20_A6_EXT: now also J507.3 (Pin_3), U505.1 (IO1)
- net SPI_MOSI: now reaches R532.1
- net SPI_MOSI_EXT: now reaches R532.2
- net SPI_MOSI_EXT: now also J506.4 (Pin_4), U503.3 (IO2)
- net IO27_A13: now reaches R546.1
- net IO21_A7_EXT: now reaches U505.3 (IO2)
- net IO21_A7_EXT: now also J507.4 (Pin_4), R542.2
- net IO24_A10_EXT: now reaches U505.4 (IO3)
- net IO24_A10_EXT: now also R543.2, J508.3 (Pin_3)
- net IO25_A11_EXT: now reaches U505.6 (IO4)
- net IO25_A11_EXT: now also R544.2, J508.4 (Pin_4)
- net IO40_A16: now reaches R547.1
- net +5V_SYS: now reaches J501.4 (Pin_4)
- net UART7_RX: now reaches R522.1
- net SPI_MISO: now reaches R533.1
- net SPI_MISO_EXT: now reaches R533.2
- net SPI_MISO_EXT: now also J506.5 (Pin_5), U503.4 (IO3)
- net IO24_A10: now reaches R543.1
- net UART7_TX: now reaches R521.1
- net VCC_GPIO_EXT: now reaches J507.1 (Pin_1)
- net VCC_GPIO_EXT: now also J508.1 (Pin_1), J509.1 (Pin_1), J510.1 (Pin_1), JP505.2 (Pin_2)
- net IO25_A11: now reaches R544.1
- net IO26_A12: now reaches R545.1
- net IO21_A7: now reaches R542.1
- net UART8_RX: now reaches R524.1
- new net +5V_EXP: JP505.3 (Pin_3)
- no-connect marks 0 -> 3
Other:
- note added: "EXTERNAL I/O | 3.3 V SIGNALS | GPIO VCC SELECTOR IS POWER ONLY"
- note added: "GPIO PORTS 1 / 2"
- note added: "GPIO PORTS 3 / 4"
- note added: "Global labels connect to Teensy. *_EXT labels are connector-side nets after 100 ohm resistors."
- note added: "I2C0 / I2C1"
- note added: "JP501-504 OPEN by default (optional 2.2k pullups) JP505: 1-2 = 3.3V default; 2-3 = 5V; ONE shunt only GPIO signals remain 3.3V. Total external 3.3V budget: 100mA."
- note added: "OPTIONS / ADDITIONAL SPI PROTECTION"
- note added: "SPI"
- note added: "UART7 / UART8"
- note removed: "Matek battery monitor / expansion I/O (1)"
- note removed: "PLACEMENT ONLY - all pins intentionally unwired; see notes in symbol properties."
- note removed: "REVIEW"
- title: Matek battery monitor / expansion I/O (1) -> External I2C / UART / SPI / GPIO 4 ports
- moved on the sheet: J501, J502, J503, J504, J505, J506, JP501, JP502, JP503, JP504, R511, R512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
