File: hardware/central-board-placement/central-board-placement.kicad_sch (KiCad schematic)
At the start: 0 parts

Commit message: Save all current circuit, firmware, CAD and manufacturing work
Other:
- note added: "ARM: GUI over USB + SW211 -> shared Teensy safety gate. E-stop release does not re-arm. A new RUN request is required after ARM. See S02B / S04. Firmware integration is separate from this schematic."
- note added: "CENTRAL BOARD / CIRCUIT DESIGN"
- note added: "Nonpower wiring added 2026-09-29. Safety TBD parts / return connection remain unresolved."
- note removed: "10 parts"
- note removed: "11 parts"
- note removed: "21 parts"
- note removed: "36 parts"
- note removed: "41 parts"
- note removed: "43 parts"
- note removed: "CENTRAL BOARD / UNWIRED COMPONENT PLACEMENT"
- note removed: "Open a sheet to wire the components. Footprints marked TBD remain unassigned."
- title: Central board - symbol placement index -> Central board - circuit index
Changed lines of the file:
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@@
 (kicad_sch
-(version 20250114)
+(version 20260306)
 (generator "eeschema")
+(generator_version "10.0")
 (paper "A3")
 (title_block
-(title "Central board - symbol placement index")
-(date "2026-09-23")
-(rev "PLACEMENT ONLY")
+(title "Central board - circuit index")
+(date "2026-09-29")
+(rev "WIRED DRAFT")
 (company "Differential Swerve")
-(comment 1 "Unwired draft - not for fabrication"))
-(text "CENTRAL BOARD / UNWIRED COMPONENT PLACEMENT"
+(comment 1 "Safety TBDs remain. Not for fabrication."))
+(text "ARM: GUI over USB + SW211 -> shared Teensy safety gate.\nE-stop release does not re-arm. A new RUN request is required after ARM.\nSee S02B / S04. Firmware integration is separate from this schematic."
+(exclude_from_sim no)
+(at 205 210 0)
+(effects
+(font
+(size 1.5 1.5)))
+)
+(text "CENTRAL BOARD / CIRCUIT DESIGN"
+(exclude_from_sim no)
 (at 205 20 0)
 (effects
@@
 (size 2.54 2.54)))
 )
-(text "Open a sheet to wire the components. Footprints marked TBD remain unassigned."
+(text "Nonpower wiring added 2026-09-29. Safety TBD parts / return connection remain unresolved."
+(exclude_from_sim no)
 (at 205 28 0)
 (effects
@@
 )
 (sheet
+(at 150 45)
+(size 110 24)
+(exclude_from_sim no)
+(in_bom yes)
+(on_board yes)
+(dnp no)
+(stroke
+(width 0.1524)
+(type solid))
+(fill
+(color 0 0 0 0))
+(property "Sheetname" "Star power / Teensy / indicators (1)"
+(at 205 42 0)
+(show_name no)
+(do_not_autoplace no)
+(effects
+(font
+(size 1.27 1.27))))
+(property "Sheetfile" "S02B_star_teensy-1.kicad_sch"
+(at 205 72 0)
+(show_name no)
+(do_not_autoplace no)
+(effects
+(font
+(size 1.27 1.27))))
+(instances
+(project "central-board-placement"
+(path "/86ff21e2-ce3a-5bf6-854a-178e7ad1d673"
+(page "3")))))
+(sheet
+(at 25 87)
+(size 110 24)
+(exclude_from_sim no)
+(in_bom yes)
+(on_board yes)
+(dnp no)
+(stroke
+(width 0.1524)
+(type solid))
+(fill
+(color 0 0 0 0))
+(property "Sheetname" "CAN2 Expansion (1)"
+(at 80 84 0)
+(show_name no)
+(do_not_autoplace no)
+(effects
+(font
+(size 1.27 1.27))))
+(property "Sheetfile" "S03_CAN2-1.kicad_sch"
+(at 80 114 0)
+(show_name no)
+(do_not_autoplace no)
+(effects
+(font
+(size 1.27 1.27))))
+(instances
+(project "central-board-placement"
+(path "/86ff21e2-ce3a-5bf6-854a-178e7ad1d673"
+(page "5")))))
+(sheet
 (at 25 45)
 (size 110 24)
+(exclude_from_sim no)
+(in_bom yes)
+(on_board yes)
+(dnp no)
 (stroke
 (width 0.1524)
@@
 (property "Sheetname" "5V input / eFuse / USB diode OR (1)"
 (at 80 42 0)
+(show_name no)
+(do_not_autoplace no)
 (effects
 (font
@@
 (property "Sheetfile" "S02A_power_input-1.kicad_sch"
 (at 80 72 0)
+(show_name no)
+(do_not_autoplace no)
 (effects
 (font
@@
 (path "/86ff21e2-ce3a-5bf6-854a-178e7ad1d673"
 (page "2")))))
-(text "21 parts"
-(at 80 57 0)
-(effects
-(font
-(size 1.27 1.27)))
-)
-(sheet
-(at 150 45)
-(size 110 24)
-(stroke
-(width 0.1524)
-(type solid))
-(fill
-(color 0 0 0 0))
-(property "Sheetname" "Star power / Teensy / indicators (1)"
-(at 205 42 0)
-(effects
-(font
-(size 1.27 1.27))))
-(property "Sheetfile" "S02B_star_teensy-1.kicad_sch"
-(at 205 72 0)
-(effects
-(font
-(size 1.27 1.27))))
-(instances
-(project "central-board-placement"
-(path "/86ff21e2-ce3a-5bf6-854a-178e7ad1d673"
-(page "3")))))
-(text "41 parts"
-(at 205 57 0)
-(effects
-(font
-(size 1.27 1.27)))
-)
+(sheet
+(at 150 87)
+(size 110 24)
+(exclude_from_sim no)
+(in_bom yes)
+(on_board yes)
+(dnp no)
+(stroke
+(width 0.1524)
+(type solid))
+(fill
+(color 0 0 0 0))
+(property "Sheetname" "CAN3 Drive (1)"
+(at 205 84 0)
+(show_name no)
+(do_not_autoplace no)
+(effects
+(font
+(size 1.27 1.27))))
+(property "Sheetfile" "S03_CAN3-1.kicad_sch"
+(at 205 114 0)
+(show_name no)
+(do_not_autoplace no)
+(effects
+(font
+(size 1.27 1.27))))
+(instances
+(project "central-board-placement"
+(path "/86ff21e2-ce3a-5bf6-854a-178e7ad1d673"
+(page "6")))))
 (sheet
 (at 275 45)
 (size 110 24)
+(exclude_from_sim no)
+(in_bom yes)
+(on_board yes)
+(dnp no)
 (stroke
 (width 0.1524)
@@
 (property "Sheetname" "CAN1 Sensor (1)"
 (at 330 42 0)
+(show_name no)
+(do_not_autoplace no)
 (effects
 (font
@@
 (property "Sheetfile" "S03_CAN1-1.kicad_sch"
 (at 330 72 0)
+(show_name no)
+(do_not_autoplace no)
 (effects
 (font
@@
 (path "/86ff21e2-ce3a-5bf6-854a-178e7ad1d673"
 (page "4")))))
-(text "10 parts"
-(at 330 57 0)
-(effects
-(font
-(size 1.27 1.27)))
-)
-(sheet
-(at 25 87)
-(size 110 24)
-(stroke
-(width 0.1524)
-(type solid))
-(fill
-(color 0 0 0 0))
-(property "Sheetname" "CAN2 Expansion (1)"
-(at 80 84 0)
-(effects
-(font
-(size 1.27 1.27))))
-(property "Sheetfile" "S03_CAN2-1.kicad_sch"
-(at 80 114 0)
-(effects
-(font
-(size 1.27 1.27))))
-(instances
-(project "central-board-placement"
-(path "/86ff21e2-ce3a-5bf6-854a-178e7ad1d673"
-(page "5")))))
-(text "11 parts"
-(at 80 99 0)
-(effects
-(font
-(size 1.27 1.27)))
-)
-(sheet
-(at 150 87)
-(size 110 24)
-(stroke
-(width 0.1524)
-(type solid))
-(fill
-(color 0 0 0 0))
-(property "Sheetname" "CAN3 Drive (1)"
-(at 205 84 0)
-(effects
-(font
-(size 1.27 1.27))))
-(property "Sheetfile" "S03_CAN3-1.kicad_sch"
-(at 205 114 0)
-(effects
-(font
-(size 1.27 1.27))))
-(instances
-(project "central-board-placement"
-(path "/86ff21e2-ce3a-5bf6-854a-178e7ad1d673"
-(page "6")))))
-(text "10 parts"
-(at 205 99 0)
-(effects
-(font
-(size 1.27 1.27)))
-)
+(sheet
+(at 25 129)
+(size 110 24)
+(exclude_from_sim no)
+(in_bom yes)
+(on_board yes)
+(dnp no)
+(stroke
+(width 0.1524)
+(type solid))
+(fill
+(color 0 0 0 0))
+(property "Sheetname" "Matek battery monitor / expansion I/O (1)"
+(at 80 126 0)
+(show_name no)
+(do_not_autoplace no)
+(effects
+(font
+(size 1.27 1.27))))
+(property "Sheetfile" "S05_io-1.kicad_sch"
+(at 80 156 0)
+(show_name no)
+(do_not_autoplace no)
+(effects
+(font
+(size 1.27 1.27))))
+(instances
+(project "central-board-placement"
+(path "/86ff21e2-ce3a-5bf6-854a-178e7ad1d673"
+(page "8")))))
 (sheet
 (at 275 87)
 (size 110 24)
+(exclude_from_sim no)
+(in_bom yes)
+(on_board yes)
+(dnp no)
 (stroke
 (width 0.1524)
@@
 (property "Sheetname" "E-stop monitoring / central coil driver (1)"
 (at 330 84 0)
+(show_name no)
+(do_not_autoplace no)
 (effects
 (font
@@
 (property "Sheetfile" "S04_safety-1.kicad_sch"
 (at 330 114 0)
+(show_name no)
+(do_not_autoplace no)
 (effects
 (font
@@
 (path "/86ff21e2-ce3a-5bf6-854a-178e7ad1d673"
 (page "7")))))
-(text "36 parts"
-(at 330 99 0)
-(effects
-(font
-(size 1.27 1.27)))
-)
-(sheet
-(at 25 129)
-(size 110 24)
-(stroke
-(width 0.1524)
-(type solid))
-(fill
-(color 0 0 0 0))
-(property "Sheetname" "Matek battery monitor / expansion I/O (1)"
-(at 80 126 0)
-(effects
-(font
-(size 1.27 1.27))))
-(property "Sheetfile" "S05_io-1.kicad_sch"
-(at 80 156 0)
-(effects
-(font
-(size 1.27 1.27))))
-(instances
-(project "central-board-placement"
-(path "/86ff21e2-ce3a-5bf6-854a-178e7ad1d673"
-(page "8")))))
-(text "43 parts"
-(at 80 141 0)
-(effects
-(font
-(size 1.27 1.27)))
-)
 (sheet_instances
 (path "/"
-(page "1"))))
+(page "1")))
+(embedded_fonts no))
