File: hardware/central-board/central-board/central-board.kicad_sch (KiCad schematic)
At the start: 2 parts, among them J3 TEENSY LEFT / 68000-224HLF + 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, J4 TEENSY RIGHT / 68000-224HLF +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

Commit message: Update project design and manufacturing artifacts
Parts:
- removed J3: TEENSY LEFT / 68000-224HLF + SOCKET, Connector_PinSocket_2.54mm:PinSocket_1x24_P2.54mm_Vertical, symbol Connector_Generic:Conn_01x24
- removed J4: TEENSY RIGHT / 68000-224HLF + SOCKET, Connector_PinSocket_2.54mm:PinSocket_1x24_P2.54mm_Vertical, symbol Connector_Generic:Conn_01x24
- added IC1: TPS259470LRPWR, TPS259470LRPWR, symbol SamacSys:TPS259470LRPWR
- added J201: TEENSY LEFT / 68000-224HLF + SOCKET, Connector_PinSocket_2.54mm:PinSocket_1x24_P2.54mm_Vertical, symbol Connector_Generic:Conn_01x24
- added J202: TEENSY RIGHT / 68000-224HLF + SOCKET, Connector_PinSocket_2.54mm:PinSocket_1x24_P2.54mm_Vertical, symbol Connector_Generic:Conn_01x24
- added J7: XT30PW-F, XT30PWF, symbol SamacSys:XT30PW-F
Connections:
- net +3V3_TEENSY: now also J201.15 (Pin_15), J202.22 (Pin_22)
- net AUX_OUTPUT_EN: now also J201.11 (Pin_11)
- net BAT_MON_ALERT_N: now also J202.13 (Pin_13)
- net CAN1_RX: now also J202.21 (Pin_21)
- net CAN1_TX: now also J202.20 (Pin_20)
- net CAN2_RX: now also J201.2 (Pin_2)
- net CAN2_TX: now also J201.3 (Pin_3)
- net CAN3_RX: now also J201.22 (Pin_22)
- net CAN3_TX: now also J201.23 (Pin_23)
- net ESTOP1_AUX_OK_N: now also J201.6 (Pin_6)
- net ESTOP2_AUX_OK_N: now also J201.7 (Pin_7)
- net ESTOP_LOOP_OK_N: now also J201.5 (Pin_5)
- net GND_CTRL: now also J201.1 (Pin_1), J202.10 (Pin_10), J202.23 (Pin_23)
- net I2C0_SCL: now also J202.17 (Pin_17)
- net I2C0_SDA: now also J202.16 (Pin_16)
- net I2C1_SCL: now also J202.14 (Pin_14)
- net I2C1_SDA: now also J202.15 (Pin_15)
- net IO20_A6: now also J202.18 (Pin_18)
- net IO21_A7: now also J202.19 (Pin_19)
- net IO24_A10: now also J201.16 (Pin_16)
- net IO25_A11: now also J201.17 (Pin_17)
- net IO26_A12: now also J201.18 (Pin_18)
- net IO27_A13: now also J201.19 (Pin_19)
- net IO40_A16: now also J202.8 (Pin_8)
- net IO41_A17: now also J202.9 (Pin_9)
- net MOTOR_PWR_EN: now also J201.4 (Pin_4)
- net MOTOR_PWR_SENSE: now also J202.12 (Pin_12)
- net PWR_5V_FAULT_N: now also J201.24 (Pin_24)
- net REARM_SW_N: now also J201.8 (Pin_8)
- net SPI_CS0_N: now also J201.12 (Pin_12)
- net SPI_CS1_N: now also J202.4 (Pin_4)
- net SPI_MISO: now also J201.14 (Pin_14)
- net SPI_MOSI: now also J201.13 (Pin_13)
- net SPI_SCK: now also J202.11 (Pin_11)
- net STATUS_G_LED: now also J201.9 (Pin_9)
- net STATUS_R_LED: now also J201.10 (Pin_10)
- net UART7_RX: now also J201.20 (Pin_20)
- net UART7_TX: now also J201.21 (Pin_21)
- net UART8_RX: now also J202.2 (Pin_2)
- net UART8_TX: now also J202.3 (Pin_3)
- new net VIN_TEENSY: J202.24 (Pin_24)
Other:
- added sheet CAN_1 (../reference-2026-09-12/CAN1_REFERENCE.kicad_sch)
- added sheet CAN_2 (../reference-2026-09-12/CAN1_SENSOR.kicad_sch)
- added sheet CAN_3 (../reference-2026-09-12/CAN3_DRIVE.kicad_sch)
- note added: "TEENSY 4.1"

Commit message: Save all current circuit, firmware, CAD and manufacturing work
Parts:
- removed IC1: TPS259470LRPWR, TPS259470LRPWR, symbol SamacSys:TPS259470LRPWR
- removed J201: TEENSY LEFT / 68000-224HLF + SOCKET, Connector_PinSocket_2.54mm:PinSocket_1x24_P2.54mm_Vertical, symbol Connector_Generic:Conn_01x24
- removed J202: TEENSY RIGHT / 68000-224HLF + SOCKET, Connector_PinSocket_2.54mm:PinSocket_1x24_P2.54mm_Vertical, symbol Connector_Generic:Conn_01x24
- removed J7: XT30PW-F, XT30PWF, symbol SamacSys:XT30PW-F
- added C211, C212: 100nF, Capacitor_SMD:C_0603_1608Metric, symbol Device:C
- added D211, D213: LTST-C190KGKT, LED_SMD:LED_0603_1608Metric, symbol Device:LED
- added D212: LTST-C190KRKT, LED_SMD:LED_0603_1608Metric, symbol Device:LED
- added J210: Teensy 4.1 socket, DifferentialSwerve:Teensy41_Socket_2x24, symbol CentralPlacement:Teensy41_Socket
- added R211, R212: 1k, Resistor_SMD:R_0603_1608Metric, symbol Device:R
- added R213: 1.5k, Resistor_SMD:R_0603_1608Metric, symbol Device:R
- added R214: 10k, Resistor_SMD:R_0603_1608Metric, symbol Device:R
- added SW211: REARM switch TBD, symbol Switch:SW_Push
Connections:
- net +3V3_TEENSY: now also C212.1, J210.15 (3.3V), J210.46 (3.3V), R214.2
- net CAN1_RX: now also J210.45 (23/A9)
- net CAN1_TX: now also J210.44 (22/A8)
- net CAN2_RX: now also J210.2 (0)
- net CAN2_TX: now also J210.3 (1)
- net CAN3_RX: now also J210.22 (30)
- net CAN3_TX: now also J210.23 (31)
- net ESTOP_LOOP_OK_N: now also J210.5 (3)
- net GND_CTRL: now also C211.2, C212.2, D211.1 (K), D212.1 (K), D213.1 (K), J210.1 (GND), J210.34 (GND), J210.47 (GND), SW211.2
- net I2C0_SCL: now also J210.41 (19/A5)
- net I2C0_SDA: now also J210.40 (18/A4)
- net I2C1_SCL: now also J210.38 (16/A2)
- net I2C1_SDA: now also J210.39 (17/A3)
- net IO20_A6: now also J210.42 (20/A6)
- net IO21_A7: now also J210.43 (21/A7)
- net IO24_A10: now also J210.16 (24/A10)
- net IO25_A11: now also J210.17 (25/A11)
- net IO26_A12: now also J210.18 (26/A12)
- net IO27_A13: now also J210.19 (27/A13)
- net IO40_A16: now also J210.32 (40/A16)
- net IO41_A17: now also J210.33 (41/A17)
- net MOTOR_PWR_EN: now also J210.4 (2)
- net PWR_5V_FAULT_N: now also J210.24 (32)
- net REARM_SW_N: now also C211.1, J210.8 (6), R214.1, SW211.1
- net SPI_CS0_N: now also J210.12 (10)
- net SPI_CS1_N: now also J210.28 (36)
- net SPI_MISO: now also J210.14 (12)
- net SPI_MOSI: now also J210.13 (11)
- net SPI_SCK: now also J210.35 (13)
- net STATUS_G_LED: now also J210.9 (7), R211.1
- net STATUS_R_LED: now also J210.10 (8), R212.2
- net UART7_RX: now also J210.20 (28)
- net UART7_TX: now also J210.21 (29)
- net UART8_RX: now also J210.26 (34)
- net UART8_TX: now also J210.27 (35)
- net VIN_TEENSY: now also J210.48 (VIN)
- new net: D211.2 (A), R211.2
- new net: D212.2 (A), R212.1
- new net: D213.2 (A), R213.2
- new net +5V_SYS: R213.1
- new net PWR_USB_FAULT_N: J210.11 (9)
- no-connect marks 4 -> 8
Other:
- removed sheet CAN_1
- removed sheet CAN_2
- removed sheet CAN_3
- added sheet 5V input / eFuse / USB diode OR (1) (power_input.kicad_sch)
- added sheet CAN1 Sensor (CAN1-1.kicad_sch)
- added sheet CAN2 Expansion (CAN2-1.kicad_sch)
- added sheet CAN3 Drive (CAN3-1.kicad_sch)
- added sheet E-stop monitoring, central coil driver (safety-1.kicad_sch)
- added sheet Matek battery monitor / expansion I/O (1) (io-1.kicad_sch)
- note added: "GPIO14/A0 RESERVED / NC"
- note added: "GPIO15/A1 RESERVED / NC"
- note added: "GPIO33 RESERVED / NC"
- note added: "GPIO37 RESERVED / NC"
- note added: "GPIO38 RESERVED / NC"
- note added: "GPIO39 RESERVED / NC"
- note added: "GPIO4 RESERVED / NC"
- note added: "GPIO5 RESERVED / NC"
- note removed: "TEENSY 4.1"
