File: hardware/central-board/central-board/central-board.kicad_pcb (KiCad board)
At the start: 2 copper layers, 2 parts, among them J3 TEENSY LEFT / 68000-224HLF + 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, J4 TEENSY RIGHT / 68000-224HLF +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

Commit message: Save all current circuit, firmware, CAD and manufacturing work
Parts:
- removed J3: TEENSY LEFT / 68000-224HLF + SOCKET, Connector_PinSocket_2.54mm:PinSocket_1x24_P2.54mm_Vertical
- removed J4: TEENSY RIGHT / 68000-224HLF + SOCKET, Connector_PinSocket_2.54mm:PinSocket_1x24_P2.54mm_Vertical
- added C102: 1uF, Capacitor_SMD:C_0603_1608Metric, F.Cu at (211.5, 100.8)
- added C103: 1uF, Capacitor_SMD:C_0603_1608Metric, F.Cu at (216.1, 100.8)
- added C105: 10nF, Capacitor_SMD:C_0603_1608Metric, F.Cu at (220.6, 100.8)
- added C106: 1uF, Capacitor_SMD:C_0603_1608Metric, F.Cu at (225.2, 100.8)
- added C107: 1uF, Capacitor_SMD:C_0603_1608Metric, F.Cu at (229.7, 100.8)
- added C108: 10nF, Capacitor_SMD:C_0603_1608Metric, F.Cu at (234.3, 100.8)
- added C211: 100nF, Capacitor_SMD:C_0603_1608Metric, F.Cu at (211.5, 130.3)
- added C212: 100nF, Capacitor_SMD:C_0603_1608Metric, F.Cu at (216.1, 130.3)
- added C311: 100nF, Capacitor_SMD:C_0603_1608Metric, F.Cu at (211.5, 164.4)
- added C312: 100nF, Capacitor_SMD:C_0603_1608Metric, F.Cu at (216.1, 164.4)
- added C313: 100nF, Capacitor_SMD:C_0603_1608Metric, F.Cu at (220.6, 164.4)
- added C314: 100nF, Capacitor_SMD:C_0603_1608Metric, F.Cu at (225.2, 164.4)
- added C315: 100nF, Capacitor_SMD:C_0603_1608Metric, F.Cu at (229.7, 164.4)
- added C316: 100nF, Capacitor_SMD:C_0603_1608Metric, F.Cu at (234.3, 164.4)
- added C401: 100nF, Capacitor_SMD:C_0603_1608Metric, F.Cu at (211.5, 189.9)
- added D101: PMEG2010EA,115, Diode_SMD:D_SOD-323, F.Cu at (238.9, 101.0)
- added D102: PMEG2010EA,115, Diode_SMD:D_SOD-323, F.Cu at (243.7, 101.0)
- added D201: LTST-C190KGKT, LED_SMD:LED_0603_1608Metric, F.Cu at (220.6, 130.3)
- added D202: LTST-C190KGKT, LED_SMD:LED_0603_1608Metric, F.Cu at (225.2, 130.3)
- added D203: LTST-C190KGKT, LED_SMD:LED_0603_1608Metric, F.Cu at (229.7, 130.3)
- added D204: LTST-C190KGKT, LED_SMD:LED_0603_1608Metric, F.Cu at (234.3, 130.3)
- added D205: LTST-C190KGKT, LED_SMD:LED_0603_1608Metric, F.Cu at (238.8, 130.3)
- added D206: LTST-C190KGKT, LED_SMD:LED_0603_1608Metric, F.Cu at (243.4, 130.3)
- added D211: LTST-C190KGKT, LED_SMD:LED_0603_1608Metric, F.Cu at (247.9, 130.3)
- added D212: LTST-C190KRKT, LED_SMD:LED_0603_1608Metric, F.Cu at (252.5, 130.3)
- added D213: LTST-C190KGKT, LED_SMD:LED_0603_1608Metric, F.Cu at (257.0, 130.3)
- added D311: ESD2CAN24DBZRQ1, Package_TO_SOT_SMD:SOT-23, F.Cu at (239.3, 165.4)
- added D312: ESD2CAN24DBZRQ1, Package_TO_SOT_SMD:SOT-23, F.Cu at (244.7, 165.4)
- added D313: ESD2CAN24DBZRQ1, Package_TO_SOT_SMD:SOT-23, F.Cu at (250.2, 165.4)
- added D401: 1N4148W, Diode_SMD:D_SOD-123, F.Cu at (216.9, 190.3)
- added F201: 1206L050/15YR, Fuse:Fuse_1206_3216Metric, F.Cu at (262.4, 130.7)
- added F202: 1206L050/15YR, Fuse:Fuse_1206_3216Metric, F.Cu at (268.5, 130.7)
- added F203: 1206L050/15YR, Fuse:Fuse_1206_3216Metric, F.Cu at (274.7, 130.7)
- added F204: 1206L050/15YR, Fuse:Fuse_1206_3216Metric, F.Cu at (280.8, 130.7)
- added F205: 1206L075/16WR, Fuse:Fuse_1206_3216Metric, F.Cu at (287.0, 130.7)
- added F206: 1206L050/15YR, Fuse:Fuse_1206_3216Metric, F.Cu at (293.1, 130.7)
- added H1: MountingHole_3.2mm_M3, MountingHole_3.2mm_M3, F.Cu at (104.0, 104.0)
- added H2: MountingHole_3.2mm_M3, MountingHole_3.2mm_M3, F.Cu at (196.0, 104.0)
- added H3: MountingHole_3.2mm_M3, MountingHole_3.2mm_M3, F.Cu at (104.0, 176.0)
- added H4: MountingHole_3.2mm_M3, MountingHole_3.2mm_M3, F.Cu at (196.0, 176.0)
- added J101: XT30PW-M, Connector_AMASS:AMASS_XT30PW-M_1x02_P2.50mm_Horizontal, F.Cu at (256.6, 113.6)
- added J201: SM02B-GHS-TB, Connector_JST:JST_GH_SM02B-GHS-TB_1x02-1MP_P1.25mm_Horizontal, F.Cu at (300.5, 132.8)
- added J202: SM02B-GHS-TB, Connector_JST:JST_GH_SM02B-GHS-TB_1x02-1MP_P1.25mm_Horizontal, F.Cu at (309.0, 132.8)
- added J203: SM02B-GHS-TB, Connector_JST:JST_GH_SM02B-GHS-TB_1x02-1MP_P1.25mm_Horizontal, F.Cu at (317.6, 132.8)
- added J204: SM02B-GHS-TB, Connector_JST:JST_GH_SM02B-GHS-TB_1x02-1MP_P1.25mm_Horizontal, F.Cu at (213.5, 140.8)
- added J210: Teensy 4.1 socket, DifferentialSwerve:Teensy41_Socket_2x24, F.Cu at (221.1, 146.8)
- added J311: SM03B-GHS-TB, Connector_JST:JST_GH_SM03B-GHS-TB_1x03-1MP_P1.25mm_Horizontal, F.Cu at (257.8, 166.9)
- added J312: SM03B-GHS-TB, Connector_JST:JST_GH_SM03B-GHS-TB_1x03-1MP_P1.25mm_Horizontal, F.Cu at (267.6, 166.9)
- added J313: SM03B-GHS-TB, Connector_JST:JST_GH_SM03B-GHS-TB_1x03-1MP_P1.25mm_Horizontal, F.Cu at (277.4, 166.9)
- added J314: SM03B-GHS-TB, Connector_JST:JST_GH_SM03B-GHS-TB_1x03-1MP_P1.25mm_Horizontal, F.Cu at (287.2, 166.9)
- added J315: SM03B-GHS-TB, Connector_JST:JST_GH_SM03B-GHS-TB_1x03-1MP_P1.25mm_Horizontal, F.Cu at (297.0, 166.9)
- added J316: SM03B-GHS-TB, Connector_JST:JST_GH_SM03B-GHS-TB_1x03-1MP_P1.25mm_Horizontal, F.Cu at (306.8, 166.9)
- added J403: TBD 2pin, Connector_JST:JST_XH_S2B-XH-A_1x02_P2.50mm_Horizontal, F.Cu at (223.8, 191.9)
- added J501: SM04B-GHS-TB, Connector_JST:JST_GH_SM04B-GHS-TB_1x04-1MP_P1.25mm_Horizontal, F.Cu at (214.8, 212.4)
- added J502: SM04B-GHS-TB, Connector_JST:JST_GH_SM04B-GHS-TB_1x04-1MP_P1.25mm_Horizontal, F.Cu at (225.8, 212.4)
- added J503: SM04B-GHS-TB, Connector_JST:JST_GH_SM04B-GHS-TB_1x04-1MP_P1.25mm_Horizontal, F.Cu at (236.9, 212.4)
- added J504: SM03B-GHS-TB, Connector_JST:JST_GH_SM03B-GHS-TB_1x03-1MP_P1.25mm_Horizontal, F.Cu at (247.3, 212.4)
- added J505: SM03B-GHS-TB, Connector_JST:JST_GH_SM03B-GHS-TB_1x03-1MP_P1.25mm_Horizontal, F.Cu at (257.1, 212.4)
- added J506: SM07B-GHS-TB, Connector_JST:JST_GH_SM07B-GHS-TB_1x07-1MP_P1.25mm_Horizontal, F.Cu at (269.4, 212.4)
- added J507: SM04B-GHS-TB, Connector_JST:JST_GH_SM04B-GHS-TB_1x04-1MP_P1.25mm_Horizontal, F.Cu at (282.3, 212.4)
- added J508: SM04B-GHS-TB, Connector_JST:JST_GH_SM04B-GHS-TB_1x04-1MP_P1.25mm_Horizontal, F.Cu at (293.4, 212.4)
- added J509: SM04B-GHS-TB, Connector_JST:JST_GH_SM04B-GHS-TB_1x04-1MP_P1.25mm_Horizontal, F.Cu at (304.4, 212.4)
- added J510: SM04B-GHS-TB, Connector_JST:JST_GH_SM04B-GHS-TB_1x04-1MP_P1.25mm_Horizontal, F.Cu at (315.4, 212.4)
- added JP501: Pullup enable N.O., Jumper:SolderJumper-2_P1.3mm_Open_RoundedPad1.0x1.5mm, F.Cu at (323.4, 210.5)
- added JP502: Pullup enable N.O., Jumper:SolderJumper-2_P1.3mm_Open_RoundedPad1.0x1.5mm, F.Cu at (211.7, 218.5)
- added JP503: Pullup enable N.O., Jumper:SolderJumper-2_P1.3mm_Open_RoundedPad1.0x1.5mm, F.Cu at (216.6, 218.5)
- added JP504: Pullup enable N.O., Jumper:SolderJumper-2_P1.3mm_Open_RoundedPad1.0x1.5mm, F.Cu at (221.5, 218.5)
- added JP505: GPIO VCC 3V3/5V select, Connector_PinHeader_2.54mm:PinHeader_1x03_P2.54mm_Vertical, F.Cu at (226.5, 219.0)
- added Q401: IRLML0100TRPBF, Package_TO_SOT_SMD:SOT-23, F.Cu at (232.8, 190.8)
- added R101: 750, Resistor_SMD:R_0603_1608Metric, F.Cu at (264.3, 100.8)
- added R102: 732k, Resistor_SMD:R_0603_1608Metric, F.Cu at (268.9, 100.8)
- added R103: 51.1k, Resistor_SMD:R_0603_1608Metric, F.Cu at (273.4, 100.8)
- added R104: 221k, Resistor_SMD:R_0603_1608Metric, F.Cu at (277.9, 100.8)
- added R105: 10k, Resistor_SMD:R_0603_1608Metric, F.Cu at (282.5, 100.8)
- added R106: 0, Resistor_SMD:R_0603_1608Metric, F.Cu at (287.1, 100.8)
- added R107: 3.32k 1%, Resistor_SMD:R_0603_1608Metric, F.Cu at (291.6, 100.8)
- added R108: 232k 1%, Resistor_SMD:R_0603_1608Metric, F.Cu at (296.1, 100.8)
- added R109: 100k 1%, Resistor_SMD:R_0603_1608Metric, F.Cu at (300.7, 100.8)
- added R110: 100k 1%, Resistor_SMD:R_0603_1608Metric, F.Cu at (305.2, 100.8)
- added R111: 37.4k 1%, Resistor_SMD:R_0603_1608Metric, F.Cu at (309.8, 100.8)
- added R112: 10k, Resistor_SMD:R_0603_1608Metric, F.Cu at (314.4, 100.8)
- added R201: 1.5k, Resistor_SMD:R_0603_1608Metric, F.Cu at (284.2, 138.3)
- added R202: 1.5k, Resistor_SMD:R_0603_1608Metric, F.Cu at (288.8, 138.3)
- added R203: 1.5k, Resistor_SMD:R_0603_1608Metric, F.Cu at (293.3, 138.3)
- added R204: 1.5k, Resistor_SMD:R_0603_1608Metric, F.Cu at (297.9, 138.3)
- added R205: 1.5k, Resistor_SMD:R_0603_1608Metric, F.Cu at (302.4, 138.3)
- added R206: 1.5k, Resistor_SMD:R_0603_1608Metric, F.Cu at (307.0, 138.3)
- added R211: 1k, Resistor_SMD:R_0603_1608Metric, F.Cu at (311.5, 138.3)
- added R212: 1k, Resistor_SMD:R_0603_1608Metric, F.Cu at (316.1, 138.3)
- added R213: 1.5k, Resistor_SMD:R_0603_1608Metric, F.Cu at (320.6, 138.3)
- added R214: 10k, Resistor_SMD:R_0603_1608Metric, F.Cu at (325.2, 138.3)
- added R311: 120, Resistor_SMD:R_0603_1608Metric, F.Cu at (313.9, 164.4)
- added R312: 120, Resistor_SMD:R_0603_1608Metric, F.Cu at (318.5, 164.4)
- added R313: 120, Resistor_SMD:R_0603_1608Metric, F.Cu at (323.0, 164.4)
- added R401: 2.2k, Resistor_SMD:R_0603_1608Metric, F.Cu at (237.8, 189.9)
- added R402: 2.2k, Resistor_SMD:R_0603_1608Metric, F.Cu at (242.4, 189.9)
- added R409: 10k, Resistor_SMD:R_0603_1608Metric, F.Cu at (246.9, 189.9)
- added R413: 100k, Resistor_SMD:R_0603_1608Metric, F.Cu at (251.5, 189.9)
- added R414: 100, Resistor_SMD:R_0603_1608Metric, F.Cu at (256.0, 189.9)
- added R415: 100k, Resistor_SMD:R_0603_1608Metric, F.Cu at (260.6, 189.9)
- added R511: 100, Resistor_SMD:R_0603_1608Metric, F.Cu at (231.3, 218.0)
- added R512: 100, Resistor_SMD:R_0603_1608Metric, F.Cu at (235.9, 218.0)
- added R513: 100, Resistor_SMD:R_0603_1608Metric, F.Cu at (240.4, 218.0)
- added R514: 100, Resistor_SMD:R_0603_1608Metric, F.Cu at (245.0, 218.0)
- added R521: 100, Resistor_SMD:R_0603_1608Metric, F.Cu at (249.5, 218.0)
- added R522: 100, Resistor_SMD:R_0603_1608Metric, F.Cu at (254.1, 218.0)
- added R523: 100, Resistor_SMD:R_0603_1608Metric, F.Cu at (258.6, 218.0)
- added R524: 100, Resistor_SMD:R_0603_1608Metric, F.Cu at (263.2, 218.0)
- added R531: 100, Resistor_SMD:R_0603_1608Metric, F.Cu at (267.7, 218.0)
- added R532: 100, Resistor_SMD:R_0603_1608Metric, F.Cu at (272.3, 218.0)
- added R533: 100, Resistor_SMD:R_0603_1608Metric, F.Cu at (276.8, 218.0)
- added R534: 100, Resistor_SMD:R_0603_1608Metric, F.Cu at (281.4, 218.0)
- added R535: 100, Resistor_SMD:R_0603_1608Metric, F.Cu at (285.9, 218.0)
- added R541: 100, Resistor_SMD:R_0603_1608Metric, F.Cu at (290.5, 218.0)
- added R542: 100, Resistor_SMD:R_0603_1608Metric, F.Cu at (295.0, 218.0)
- added R543: 100, Resistor_SMD:R_0603_1608Metric, F.Cu at (299.6, 218.0)
- added R544: 100, Resistor_SMD:R_0603_1608Metric, F.Cu at (304.1, 218.0)
- added R545: 100, Resistor_SMD:R_0603_1608Metric, F.Cu at (308.7, 218.0)
- added R546: 100, Resistor_SMD:R_0603_1608Metric, F.Cu at (313.2, 218.0)
- added R547: 100, Resistor_SMD:R_0603_1608Metric, F.Cu at (317.8, 218.0)
- added R548: 100, Resistor_SMD:R_0603_1608Metric, F.Cu at (322.3, 218.0)
- added R551: 2.2k, Resistor_SMD:R_0603_1608Metric, F.Cu at (326.9, 218.0)
- added R552: 2.2k, Resistor_SMD:R_0603_1608Metric, F.Cu at (211.5, 228.2)
- added R553: 2.2k, Resistor_SMD:R_0603_1608Metric, F.Cu at (216.1, 228.2)
- added R554: 2.2k, Resistor_SMD:R_0603_1608Metric, F.Cu at (220.6, 228.2)
- added SW311: JS102011SAQN, DifferentialSwerve:JS102011SAQN, F.Cu at (215.6, 177.2)
- added SW312: JS102011SAQN, DifferentialSwerve:JS102011SAQN, F.Cu at (228.3, 177.2)
- added SW313: JS102011SAQN, DifferentialSwerve:JS102011SAQN, F.Cu at (241.0, 177.2)
- added TP101: +5V_RAW, DifferentialSwerve:Harwin_S1751-46R, F.Cu at (319.2, 101.1)
- added TP102: +5V_SYS, DifferentialSwerve:Harwin_S1751-46R, F.Cu at (324.5, 101.1)
- added TP401: ESTOP_LOOP_OK_N, TestPoint:TestPoint_Pad_D1.5mm, F.Cu at (264.9, 190.4)
- added TP406: GND_CTRL_LED, TestPoint:TestPoint_Pad_D1.5mm, F.Cu at (269.0, 190.4)
- added TP501: GND_CTRL, DifferentialSwerve:Harwin_S1751-46R, F.Cu at (225.5, 228.5)
- added U101: TPS259470LRPWR, DifferentialSwerve:TPS25947_RPW_10Pin, F.Cu at (212.3, 119.7)
- added U102: TPS259470ARPWR, DifferentialSwerve:TPS25947_RPW_10Pin, F.Cu at (218.4, 119.7)
- added U311: TCAN1051VDRQ1, Package_SO:SOIC-8_3.9x4.9mm_P1.27mm, F.Cu at (251.8, 174.3)
- added U312: TCAN1051VDRQ1, Package_SO:SOIC-8_3.9x4.9mm_P1.27mm, F.Cu at (260.8, 174.3)
- added U313: TCAN1051VDRQ1, Package_SO:SOIC-8_3.9x4.9mm_P1.27mm, F.Cu at (269.8, 174.3)
- added U401: LTV-817S, Package_DIP:SMDIP-4_W9.53mm, F.Cu at (277.8, 191.9)
- added U402: SN74AHCT1G125DBVR, Package_TO_SOT_SMD:SOT-23-5, F.Cu at (287.5, 190.8)
- added U501: SRV05-4, Package_TO_SOT_SMD:SOT-23-6, F.Cu at (231.0, 229.1)
- added U502: SRV05-4, Package_TO_SOT_SMD:SOT-23-6, F.Cu at (236.7, 229.1)
- added U503: SRV05-4, Package_TO_SOT_SMD:SOT-23-6, F.Cu at (242.4, 229.1)
- added U504: SRV05-4, Package_TO_SOT_SMD:SOT-23-6, F.Cu at (248.1, 229.1)
- added U505: SRV05-4, Package_TO_SOT_SMD:SOT-23-6, F.Cu at (253.8, 229.1)
- added U506: SRV05-4, Package_TO_SOT_SMD:SOT-23-6, F.Cu at (259.4, 229.1)
Other:
- board outline added: 100 x 80 mm

Commit message: Select X402 ground net tie and save central board updates
Parts:
- added D405: SMBJ33CA, Diode_SMD:D_SMB, F.Cu at (101.0, 142.4)
- added J401: TBD E-stop 4pin, Connector_JST:JST_XH_S4B-XH-A_1x04_P2.50mm_Horizontal, F.Cu at (118.0, 115.4)
- added X402: NetTie_3, NetTie:NetTie-3_SMD_Pad2.0mm, F.Cu at (91.3, 141.1)
- moved C311 755.3 mm to (-399.4, -279.8)
- moved C312 755.3 mm to (-394.8, -279.8)
- moved D311 755.3 mm to (-371.6, -278.9)
- moved J311 755.3 mm to (-353.1, -277.4)
- moved J312 755.3 mm to (-343.3, -277.4)
- moved R311 755.3 mm to (-297.0, -279.8)
- moved SW311 755.3 mm to (-395.3, -267.0)
- moved U311 755.3 mm to (-359.1, -269.9)
- moved C313 736.8 mm to (-509.3, 63.9)
- moved C314 736.8 mm to (-504.7, 63.9)
- moved D312 736.8 mm to (-485.2, 64.8)
- moved J313 736.8 mm to (-452.5, 66.3)
- moved J314 736.8 mm to (-442.7, 66.3)
- moved R312 736.8 mm to (-411.4, 63.9)
- moved U312 736.8 mm to (-469.1, 73.8)
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Other:
- board size 100 x 80 mm -> 90 x 50 mm
